File: kicad_source/OpenCyphalServoController12.kicad_pcb (KiCad board)
At the start: 2 copper layers, 52 x 36 mm, 63 parts, among them CN1 RASPBERRYPI_PICO, CN11 CONN_02X03, CN12 Conn_01x03, CN2 SM04B-SRSS-TB, CN3 SM04B-SRSS-TB, CN4 GH_SM04B-GHS-TB, CN5 GH_SM04B-GHS-TB, CN6 691322310002, CN7 CONN_02X03, CN8 Conn_02x08_Odd_Even, SW1 SPST, U3 24LC64, U8 MCP2515, U9 SN65HVD232, Y1 16MHz

Commit message: started first placement
Parts:
- removed U8: MCP2515, Package_SO:SOIC-18W_7.5x11.6mm_P1.27mm
- removed U9: SN65HVD232, Package_SO:SOIC-8_3.9x4.9mm_P1.27mm
- added C13: 100 uF / 50 V, Capacitor_SMD:CP_Elec_8x10, F.Cu at (98.0, 105.5)
- added C14: 100 nF, Capacitor_SMD:C_0603_1608Metric, F.Cu at (90.0, 66.5)
- added C15: 100 uF / 50 V, Capacitor_SMD:CP_Elec_8x10, F.Cu at (74.5, 58.5)
- added C16: 4.7uF 50V, Capacitor_SMD:C_1210_3225Metric, F.Cu at (93.5, 67.0)
- added C17: 100 nF, Capacitor_SMD:C_0603_1608Metric, F.Cu at (92.5, 64.5)
- added C18: 1000 uF / 10 V, Capacitor_SMD:CP_Elec_8x10, F.Cu at (130.0, 64.5)
- added C20: 47uF 10V, Capacitor_SMD:C_1210_3225Metric, F.Cu at (92.5, 62.0)
- added C21: 1000 uF / 10 V, Capacitor_SMD:CP_Elec_8x10, F.Cu at (126.5, 98.5)
- added C22: 47uF 10V, Capacitor_SMD:C_1210_3225Metric, F.Cu at (92.5, 58.5)
- added C23: 47uF 10V, Capacitor_SMD:C_1210_3225Metric, F.Cu at (92.5, 55.0)
- added CN10: GH_SM04B-GHS-TB, Connector_JST:JST_GH_SM04B-GHS-TB_1x04-1MP_P1.25mm_Horizontal, F.Cu at (64.0, 90.0)
- added CN13: DNI, Connector_Phoenix_MC:PhoenixContact_MC_1,5_2-G-3.5_1x02_P3.50mm_Horizontal, F.Cu at (65.9, 61.8)
- added CN14: DNI, Connector_PinHeader_2.54mm:PinHeader_1x02_P2.54mm_Vertical, F.Cu at (109.3, 101.0)
- added CN9: RASPBERRYPI_PICO, generationmake:RASPI_PICO_SOLDER_Kopie, F.Cu at (116.5, 81.5)
- added D1: LED red, LED_SMD:LED_0603_1608Metric, F.Cu at (140.5, 101.0)
- added D3: MBR0530T1G, Diode_SMD:D_SOD-123, F.Cu at (72.0, 87.0)
- added D6: MBR0530T1G, Diode_SMD:D_SOD-123, F.Cu at (84.5, 88.0)
- added L4: 7443251000 (10 uH), Inductor_SMD:L_Wuerth_HCI-1050, F.Cu at (84.5, 59.0)
- added R26: 120k, Resistor_SMD:R_0603_1608Metric, F.Cu at (86.5, 74.0)
- added R27: 20k, Resistor_SMD:R_0603_1608Metric, F.Cu at (85.0, 74.0)
- added R28: 10k, Resistor_SMD:R_0603_1608Metric, F.Cu at (88.0, 74.0)
- added R29: 1R, Resistor_SMD:R_0603_1608Metric, F.Cu at (90.0, 70.0)
- added R30: 30k, Resistor_SMD:R_0603_1608Metric, F.Cu at (82.0, 74.0)
- added R31: 120k, Resistor_SMD:R_0603_1608Metric, F.Cu at (81.5, 66.5)
- added R32: 20k, Resistor_SMD:R_0603_1608Metric, F.Cu at (81.5, 68.0)
- added R33: 2k2, Resistor_SMD:R_0603_1608Metric, F.Cu at (88.0, 108.5)
- added U1: 24LC64, Package_SO:SOIC-8_3.9x4.9mm_P1.27mm, F.Cu at (99.0, 65.0)
- added U2: MCP2515, Package_SO:SOIC-18W_7.5x11.6mm_P1.27mm, F.Cu at (79.0, 101.0)
- added U4: RAA211650, Package_DFN_QFN:QFN-28-1EP_4x5mm_P0.5mm_EP2.65x3.65mm, F.Cu at (86.5, 68.5)
- C10: value 100nF -> 4.7uF 50V; footprint Capacitor_SMD:C_0603_1608Metric -> Capacitor_SMD:C_1210_3225Metric
- C11: value 100 uF / 6,3 V -> 1 uF; footprint Capacitor_SMD:CP_Elec_5x5.3 -> Capacitor_SMD:C_0603_1608Metric
- C12: value 100 uF / 6,3 V -> 2.2 uF; footprint Capacitor_SMD:CP_Elec_5x5.3 -> Capacitor_SMD:C_0603_1608Metric
- C6: value 100nF -> 10pF
- C8: value 10pF -> 100nF
- C9: value 100nF -> 10nF
- CN1: value RASPBERRYPI_PICO -> SM04B-SRSS-TB; footprint generationmake:RASPI_PICO_SOLDER_Kopie -> Connector_JST:JST_SH_SM04B-SRSS-TB_1x04-1MP_P1.00mm_Horizontal; moved to F.Cu
- CN11: value CONN_02X03 -> GH_SM04B-GHS-TB; footprint Connector_PinHeader_2.54mm:PinHeader_2x03_P2.54mm_Vertical -> Connector_JST:JST_GH_SM04B-GHS-TB_1x04-1MP_P1.25mm_Horizontal
- CN12: value Conn_01x03 -> Powerpole_2; footprint Connector_JST:JST_PH_S3B-PH-SM4-TB_1x03-1MP_P2.00mm_Horizontal -> generationmake:POWERPOLE_hor_2
- CN2, CN3: value SM04B-SRSS-TB -> CONN_02X03; footprint Connector_JST:JST_SH_SM04B-SRSS-TB_1x04-1MP_P1.00mm_Horizontal -> Connector_PinHeader_2.54mm:PinHeader_2x03_P2.54mm_Horizontal
- CN4, CN5: value GH_SM04B-GHS-TB -> CONN_02X03; footprint Connector_JST:JST_GH_SM04B-GHS-TB_1x04-1MP_P1.25mm_Horizontal -> Connector_PinHeader_2.54mm:PinHeader_2x03_P2.54mm_Horizontal
- CN6: value 691322310002 -> CONN_02X03; footprint CON_wuerth:WR-TBL_691322310002 -> Connector_PinHeader_2.54mm:PinHeader_2x03_P2.54mm_Horizontal
- CN8: value Conn_02x08_Odd_Even -> SM04B-SRSS-TB; footprint Connector_PinHeader_2.54mm:PinHeader_2x08_P2.54mm_Vertical -> Connector_JST:JST_SH_SM04B-SRSS-TB_1x04-1MP_P1.00mm_Horizontal
- D2: value MBR0530T1G -> LED yellow; footprint Diode_SMD:D_SOD-123 -> LED_SMD:LED_0603_1608Metric
- D4: value LED yellow -> SMCJ40A; footprint LED_SMD:LED_0603_1608Metric -> Diode_SMD:D_SMC
- D5: value LED red -> LED green
- R1, R10, R14, R2, R3, R4, R5, R6, R9: value 10k -> 100R
- R13: value 100k -> 100R
- R15: value 3k3 -> 100k
- R16: value 3k3 -> 10k
- R17: value 10k -> 100k
- R19: value 10k -> 3k3
- R20: value 100R -> 100k
- R21, R23, R24, R25: value 100R -> 10k
- R22: value 100R -> 3k3
- U3: value 24LC64 -> SN65HVD232
- moved L2 70.9 mm to (19.0, 117.6)
- moved L1 70.9 mm to (20.5, 124.1)
- moved D2 69.7 mm to (140.5, 96.0)
- moved L3 64.8 mm to (36.0, 120.5)
- moved CN3 64.4 mm to (116.0, 58.0), turned to 90 degrees
- moved CN8 59.6 mm to (139.0, 64.0)
- moved R22 59.3 mm to (138.5, 96.0)
- moved CN4 55.3 mm to (107.0, 58.0), turned to 90 degrees
- moved CN6 54.0 mm to (121.0, 105.0), turned to -90 degrees
- moved R14 50.9 mm to (132.5, 101.0), turned to 90 degrees
- moved CN11 48.8 mm to (64.0, 99.5)
- moved R6 48.1 mm to (134.5, 101.0), turned to -90 degrees
- moved CN5 47.7 mm to (112.0, 105.0)
- moved R19 47.6 mm to (138.5, 101.0)
- moved R2 43.9 mm to (115.0, 62.0)
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Connections:
- C1 pad 1: /INPUT0 -> +3V3
- C10 pad 1: /INPUT3 -> +BATT
- C11 pad 1: +BATT -> GND
- C11 pad 2: GND -> /Power/AVCC
- C12 pad 1: +BATT -> GND
- C12 pad 2: GND -> /Power/PVCC
- C2 pad 1: /INPUT1 -> /MEAS_CANVCC
- C3 pad 1: +3V3 -> /MEAS_BATT
- C4 pad 1: +3V3 -> /MEAS_5V
- C5 pad 1: /INPUT2 -> +3V3
- C6 pad 1: +3V3 -> /MCP2515/MCP2515_OSC2
- C7 pad 1: /MCP2515/MCP2515_OSC2 -> /MCP2515/MCP2515_OSC1
- C8 pad 1: /MCP2515/MCP2515_OSC1 -> +3V3
- C9 pad 1: /+BATT_MEAS -> GND
- C9 pad 2: GND -> /Power/SS
- CN1 pad 1: /SER_TX -> GND
- CN1 pad 2: /SER_RX -> +3V3
- CN1 pad 3: GND -> /I2C_SDA
- CN1 pad 4: unconnected-(CN1-Pad4) -> /I2C_SCL
- CN11 pad 1: /NEOPIXEL_R -> CANVCC
- CN11 pad 2: /RESERVED0_R -> /MCP2515/CANH
- CN11 pad 3: +BATT -> /MCP2515/CANL
- CN11 pad 4: +3V3 -> GND
- CN12 pad 1: /NEOPIXEL_R -> +BATT
- CN12 pad 2: +BATT -> GND
- CN2 pad 1: GND -> /SERVO01_R
- CN2 pad 2: +3V3 -> /SERVO00_R
- CN2 pad 3: /I2C_SDA -> VCC
- CN2 pad 4: /I2C_SCL -> VCC
- CN3 pad 1: GND -> /SERVO03_R
- CN3 pad 2: +3V3 -> /SERVO02_R
- CN3 pad 3: /SER_TX -> VCC
- CN3 pad 4: /SER_RX -> VCC
- CN4 pad 1: /MCP2515/CANVCC -> /SERVO05_R
- CN4 pad 2: /MCP2515/CANH -> /SERVO04_R
- CN4 pad 3: /MCP2515/CANL -> VCC
- CN4 pad 4: GND -> VCC
- CN5 pad 1: /MCP2515/CANVCC -> /SERVO07_R
- CN5 pad 2: /MCP2515/CANH -> /SERVO06_R
- CN5 pad 3: /MCP2515/CANL -> VCC
- CN5 pad 4: GND -> VCC
- CN6 pad 1: +BATT -> /SERVO09_R
- CN6 pad 2: GND -> /SERVO08_R
- CN7 pad 1: /SERVO1_R -> /SERVO11_R
- CN7 pad 2: /SERVO0_R -> /SERVO10_R
- CN7 pad 3: +BATT -> VCC
- CN7 pad 4: +BATT -> VCC
- CN8 pad 1: /ANALOG_INPUT1_R -> GND
- CN8 pad 2: GND -> +3V3
- CN8 pad 3: /ANALOG_INPUT0_R -> /SER_TX
- CN8 pad 4: GND -> /SER_RX
- D2 pad 1: Net-(D2-Pad1) -> GND
- D2 pad 2: /MCP2515/CANVCC -> /LED3_R
- D4 pad 1: GND -> +BATT
- D4 pad 2: /LED3_R -> GND
- D5 pad 2: /LED2_R -> Net-(D5-Pad2)
- F1 pad 1: +BATT -> +5V
- F1 pad 2: Net-(D2-Pad1) -> Net-(D3-Pad1)
- R1 pad 1: +3V3 -> /SERVO01
- R1 pad 2: MCP2515_INT -> /SERVO01_R
- R10 pad 1: +3V3 -> /SERVO02_R
- R10 pad 2: /I2C_SDA -> /SERVO02
- R11 pad 1: /SERVO1 -> /SERVO04_R
- R11 pad 2: /SERVO1_R -> /SERVO04
- R12 pad 1: /SERVO0_R -> /SERVO06_R
- R12 pad 2: /SERVO0 -> /SERVO06
- R13 pad 1: +BATT -> /SERVO08_R
- R13 pad 2: /+BATT_MEAS -> /SERVO08
- R14 pad 1: /+BATT_MEAS -> /SERVO10_R
- R14 pad 2: GND -> /SERVO10
- R15 pad 1: /LED3 -> CANVCC
- R15 pad 2: /LED3_R -> /MEAS_CANVCC
- R16 pad 1: /LED2 -> /MEAS_CANVCC
- R16 pad 2: /LED2_R -> GND
- R17 pad 1: /INPUT1_R -> +BATT
- R17 pad 2: /INPUT1 -> /MEAS_BATT
- R18 pad 1: /INPUT2_R -> /MEAS_BATT
- R18 pad 2: /INPUT2 -> GND
- R19 pad 1: /INPUT3_R -> /LED2
- R19 pad 2: /INPUT3 -> /LED2_R
- R2 pad 1: +3V3 -> /SERVO03
- R2 pad 2: MCP2515_CS -> /SERVO03_R
- R20 pad 1: /OUTPUT0_R -> VCC
- R20 pad 2: /OUTPUT0 -> /MEAS_5V
- R21 pad 1: /OUTPUT1_R -> /MEAS_5V
- R21 pad 2: /OUTPUT1 -> GND
- R22 pad 1: /ANALOG_INPUT0_R -> /LED3
- R22 pad 2: /ANALOG_INPUT0 -> /LED3_R
- R23 pad 1: /ANALOG_INPUT1_R -> +3V3
- R23 pad 2: /ANALOG_INPUT1 -> MCP2515_INT
- R24 pad 1: /RESERVED0_R -> +3V3
- R24 pad 2: /RESERVED0 -> MCP2515_CS
- R25 pad 1: /NEOPIXEL_R -> +3V3
- R25 pad 2: /NEOPIXEL -> /MCP2515/MCP2515_RESET
- R3 pad 1: +3V3 -> /SERVO05
- R3 pad 2: /MCP2515/MCP2515_RESET -> /SERVO05_R
- R4 pad 1: +3V3 -> /SERVO07
- R4 pad 2: /INPUT0_R -> /SERVO07_R
- R5 pad 1: +3V3 -> /SERVO09
- R5 pad 2: /INPUT1_R -> /SERVO09_R
- R6 pad 1: +3V3 -> /SERVO11
- R6 pad 2: /INPUT2_R -> /SERVO11_R
- R7 pad 2: /INPUT3_R -> /I2C_SCL
- R8 pad 1: /INPUT0_R -> +3V3
- R8 pad 2: /INPUT0 -> /I2C_SDA
- R9 pad 1: +3V3 -> /SERVO00_R
- R9 pad 2: /I2C_SCL -> /SERVO00
- U3 pad 1: GND -> /MCP2515/TXCAN
- U3 pad 3: GND -> +3V3
- U3 pad 4: GND -> /MCP2515/RXCAN
- U3 pad 5: /I2C_SDA -> unconnected-(U3-Pad5)
- U3 pad 6: /I2C_SCL -> /MCP2515/CANL
- U3 pad 7: GND -> /MCP2515/CANH
- U3 pad 8: +3V3 -> GND
Routing:
- net +BATT: track 123.7 -> 0.00 mm, vias 4 -> 0
- net GND: track 118.0 -> 0.00 mm, vias 20 -> 0
- net +3V3: track 113.3 -> 0.23 mm, vias 4 -> 0
- net /I2C_SDA: track 46.8 -> 0.00 mm, vias 1 -> 0
- net MCP2515_CS: track 46.6 -> 0.00 mm, vias 1 -> 0
- net MISO: track 44.9 -> 0.00 mm, vias 1 -> 0
- net /I2C_SCL: track 37.2 -> 0.00 mm, vias 1 -> 0
- net MCP2515_INT: track 34.4 -> 0.00 mm, vias 1 -> 0
- net /SER_TX: track 27.8 -> 0.00 mm, vias 1 -> 0
- net /SER_RX: track 27.0 -> 0.00 mm, vias 1 -> 0
- net /MCP2515/CANH: track 25.4 -> 0.00 mm
- net /ANALOG_INPUT0: track 25.1 -> 0.00 mm, vias 1 -> 0
- net SCK: track 24.3 -> 0.00 mm, vias 1 -> 0
- net /SERVO1: track 24.1 -> 0.00 mm, vias 1 -> 0
- net MOSI: track 23.8 -> 0.00 mm, vias 1 -> 0
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Other:
- board size 52 x 36 mm -> 81 x 57 mm
